Commit message: add gazebo view
currently development

File: limo_description/urdf/limo_ackerman.xacro (robot description, xacro)
@@ -4,22 +4,12 @@
     <xacro:include filename="$(find limo_description)/urdf/limo_xacro.xacro" />
     <xacro:include filename="$(find limo_description)/urdf/limo_steering_hinge.xacro" />
-    <xacro:include filename="$(find limo_description)/urdf/limo_ackerman.gazebo" />
-    <!-- Variables -->
-    <xacro:property name="M_PI" value="3.14159"/>
-    <!-- Vehicle Geometries -->
-    <xacro:property name="base_x_size" value="0.13" />
-    <xacro:property name="base_y_size" value="0.12" />
-    <xacro:property name="base_z_size" value="0.10" />
-    <xacro:property name="wheelbase" value="0.2"/>
-    <xacro:property name="track" value="0.14"/>
-    <xacro:property name="wheel_vertical_offset" value="-0.100998" />
-    <xacro:property name="base_mass" value="2.1557"/>
-    <xacro:property name="wheel_length" value="0.045" />
-    <xacro:property name="wheel_radius" value="0.045" />
+    <xacro:include filename="$(find limo_description)/urdf/inertial_macros.xacro" />
+    <xacro:include filename="$(find limo_description)/urdf/properties.xacro" />
+    <xacro:include filename="$(find limo_description)/urdf/gazbo_control.xacro" />
     <link name="base_footprint"/>
     <joint name="base_joint" type="fixed">
-    <parent link="base_footprint"/>
-    <child link="base_link"/>
-    <origin xyz="0.0 0.0 0.15" rpy="0 0 0"/>
+        <parent link="base_footprint"/>
+        <child link="base_link"/>
+        <origin xyz="0.0 0.0 0.15" rpy="0 0 0"/>
     </joint>
     <!-- Base link -->
@@ -37,4 +27,5 @@
           </geometry>
         </collision>
+        <xacro:box_inertial_matrix  m="${base_mass}" w="${base_x_size}" l="${base_y_size}" h="${base_z_size}" />
     </link>
     <link name="inertial_link">
@@ -61,4 +52,5 @@
         <origin xyz="0.0 0 -0.1" rpy="0 0 0"/>
     </xacro:limo_imu>
+    <!-- Front Wheel -->
     <xacro:limo_left_steering_hinge parent_prefix="base_link" wheel_prefix="left_steering_hinge">
         <origin xyz="${wheelbase/2} ${track/2} ${wheel_vertical_offset}" rpy="0 0  0" />
@@ -67,4 +59,5 @@
         <origin xyz="${wheelbase/2} ${-track/2} ${wheel_vertical_offset}" rpy="${M_PI} 0 0" />
     </xacro:limo_right_steering_hinge>
+    <!-- Back Wheel -->
     <link name="rear_left_wheel_link">
         <inertial>
@@ -85,4 +78,5 @@
           </geometry>
         </collision>
+        <xacro:cylinder_inertial_matrix  m="${wheel_mass}" r="${wheel_radius}" h="${wheel_length}"/>
     </link>
     <joint name="rear_left_wheel" type="continuous">
@@ -110,4 +104,5 @@
               </geometry>
             </collision>
+            <xacro:cylinder_inertial_matrix  m="${wheel_mass}" r="${wheel_radius}" h="${wheel_length}"/>
         </link>
     <joint name="rear_right_wheel" type="continuous">

File: limo_description/urdf/limo_steering_hinge.xacro (robot description, xacro)
@@ -4,4 +4,5 @@
 um die Erstellung von Steuerscharnier des Wagens zu ermöglichen. Durch Macrofunktion dient es einfach beim Aufruf in limo_base.-->
 <robot name="limo_steering_hinge" xmlns:xacro="http://www.ros.org/wiki/xacro">
+    <xacro:include filename="$(find limo_description)/urdf/inertial_macros.xacro" />
     <xacro:macro name="limo_left_steering_hinge" params="parent_prefix wheel_prefix *joint_pose">
         <link name="${wheel_prefix}">
@@ -26,4 +27,14 @@
             </collision>
         </link>
+        <transmission name="${wheel_prefix}_hinge_trans" type="SimpleTransmission">
+            <type>transmission_interface/SimpleTransmission</type>
+            <actuator name="${wheel_prefix}_hinge_motor">
+                <hardwareInterface>hardware_interface/EffortJointInterface</hardwareInterface>
+                <mechanicalReduction>1</mechanicalReduction>
+            </actuator>
+            <joint name="${wheel_prefix}_steer_joint">
+                <hardwareInterface>hardware_interface/EffortJointInterface</hardwareInterface>
+            </joint>
+        </transmission>
         <joint name="${wheel_prefix}_steering" type="revolute">
             <parent link="${parent_prefix}"/>
@@ -52,4 +63,5 @@
                 </geometry>
             </collision>
+            <xacro:cylinder_inertial_matrix  m="${wheel_mass}" r="${wheel_radius}"  h="${wheel_length}" />
         </link>
         <joint name="front_left_wheel" type="continuous">
@@ -85,5 +97,5 @@
             <xacro:insert_block name="joint_pose"/>
             <axis xyz="0 0 -1"/>
-            <limit lower="-0.523598767" upper="0.523598767" effort="5" velocity="0.5" />
+            <limit lower="-0.6" upper="0.6" effort="20" velocity="2.0"/> <!-- Increased limits -->
             <dynamics damping="1.0" friction="2.0"/>
         </joint>
@@ -106,4 +118,5 @@
                 </geometry>
             </collision>
+            <xacro:cylinder_inertial_matrix  m="${wheel_mass}" r="${wheel_radius}"  h="${wheel_length}" />
         </link>
         <joint name="front_right_wheel" type="continuous">

File: limo_description/urdf/limo_xacro.xacro (robot description, xacro)
@@ -1,5 +1,5 @@
 <?xml version="1.0"?>
 <robot name="limo_xacro" xmlns:xacro="http://ros.org/wiki/xacro">
-    <xacro:macro name="limo_wheel" params="parent_prefix wheel_prefix reflect *joint_pose">
+    <!-- <xacro:macro name="limo_wheel" params="parent_prefix wheel_prefix reflect *joint_pose">
         <link name="${wheel_prefix}_wheel_link">
             <inertial>
@@ -27,5 +27,5 @@
             <axis xyz="0 ${reflect*1} 0"/>
         </joint>
-    </xacro:macro>
+    </xacro:macro> -->
     <xacro:macro name="limo_laser" params="parent_prefix frame_prefix *joint_pose">
         <link name='${frame_prefix}_link'>
@@ -66,4 +66,36 @@
         <gazebo reference="${frame_prefix}_link">
             <material>Gazebo/Yellow</material>
+            <sensor type="ray" name="laser_sensor">
+              <pose>0 0 0 0 0 0</pose>
+              <visualize>false</visualize>
+              <update_rate>8</update_rate>
+              <ray>
+                <scan>
+                  <horizontal>
+                    <samples>720</samples>
+                    <resolution>1</resolution>
+                    <min_angle>-2.09439504</min_angle>
+                    <max_angle>2.09439504</max_angle>
+                  </horizontal>
+                </scan>
+                <range>
+                  <min>0.05</min>
+                  <max>8.0</max>
+                  <resolution>0.01</resolution>
+                </range>
+                <noise>
+                  <type>gaussian</type>
+                  <mean>0.0</mean>
+                  <stddev>0.01</stddev>
+                </noise>
+              </ray>
+              <plugin name="gazebo_ros_laser_sensor" filename="libgazebo_ros_ray_sensor.so">
+              <ros>
+                <remapping>~/out:=scan</remapping>
+              </ros>
+                <topicName>/limo/scan</topicName>
+                <frameName>laser_link</frameName>
+              </plugin>
+            </sensor>
         </gazebo>
     </xacro:macro>
@@ -112,4 +144,49 @@
         <gazebo reference="${frame_prefix}_link">
             <material>Gazebo/Yellow</material>
+            <sensor name="sensor_camera" type="depth">
+                <pose>0.0 0.0 0.0 0.0 0.0 0.0</pose>
+                <always_on>true</always_on>
+                <visualize>true</visualize>
+                <update_rate>10.0</update_rate>
+                <camera name="head">
+                <horizontal_fov>1.3962634</horizontal_fov>
+                <image>
+                    <width>640</width>
+                    <height>480</height>
+                    <format>R8G8B8</format>
+                </image>
+                <clip>
+                    <near>0.02</near>
+                    <far>300</far>
+                </clip>
+                </camera>
+                <plugin name="gazebo_ros_depth_camera_sensor" filename="libgazebo_ros_openni_kinect.so">
+                <baseline>0.2</baseline>
+                <alwaysOn>true</alwaysOn>
+                <!-- Keep this zero, update_rate in the parent <sensor> tag
+                    will control the frame rate. -->
+                <updateRate>0.0</updateRate>
+                <cameraName>camera_ir</cameraName>
+                <imageTopicName>/limo/color/image_raw</imageTopicName>
+                <cameraInfoTopicName>/limo/color/camera_info</cameraInfoTopicName>
+                <depthImageTopicName>/limo/depth/image_raw</depthImageTopicName>
+                <depthImageCameraInfoTopicName>/limo/depth/camera_info</depthImageCameraInfoTopicName>
+                <pointCloudTopicName>/limo/depth/points</pointCloudTopicName>
+                <frameName>depth_link</frameName>
+                <cameraname>depth_camera_link</cameraname>
+                <pointCloudCutoff>0.5</pointCloudCutoff>
+                <pointCloudCutoffMax>3.0</pointCloudCutoffMax>
+                <distortionK1>0</distortionK1>
+                <distortionK2>0</distortionK2>
+                <distortionK3>0</distortionK3>
+                <distortionT1>0</distortionT1>
+                <distortionT2>0</distortionT2>
+                <CxPrime>0</CxPrime>
+                <Cx>0</Cx>
+                <Cy>0</Cy>
+                <focalLength>0</focalLength>
+                <hackBaseline>0</hackBaseline>
+                </plugin>
+            </sensor>
         </gazebo>
     </xacro:macro>
@@ -152,4 +229,21 @@
         <gazebo reference="${frame_prefix}_link">
             <material>Gazebo/Yellow</material>
+            <gravity>true</gravity>
+            <sensor name="imu_sensor" type="imu">
+                <always_on>true</always_on>
+                <update_rate>100</update_rate>
+                <visualize>true</visualize>
+                <topic>__default_topic__</topic>
+                <plugin filename="libgazebo_ros_imu_sensor.so" name="imu_plugin">
+                    <topicName>/limo/imu</topicName>
+                    <bodyName>${frame_prefix}_link</bodyName>
+                    <updateRateHZ>100.0</updateRateHZ>
+                    <gaussianNoise>0.001</gaussianNoise>
+                    <xyzOffset>0 0 0</xyzOffset>
+                    <rpyOffset>0 0 0</rpyOffset>
+                    <frameName>imu_link</frameName>
+                </plugin>
+                <pose>0 0 0 0 0 0</pose>
+            </sensor>
         </gazebo>
     </xacro:macro>
