Commit message: update odom and lab1.3

File: limo_description/urdf/limo_ackerman.urdf.xacro (robot description, xacro)
@@ -47,7 +47,8 @@
         <origin xyz="0.103 0 -0.034" rpy="0 0 0"/>
     </xacro:limo_laser> -->
-    <xacro:limo_depth_camera parent_prefix="base_link" frame_prefix="depth_camera">
+    <!-- <xacro:limo_depth_camera parent_prefix="base_link" frame_prefix="depth_camera">
         <origin xyz="0.084 0 0.026" rpy="0 0 0"/>
     </xacro:limo_depth_camera>
+     -->
     <xacro:limo_imu parent_prefix="base_link" frame_prefix="imu">
         <origin xyz="0.0 0 -0.1" rpy="0 0 0"/>

File: limo_description/urdf/limo_xacro.xacro (robot description, xacro)
@@ -336,3 +336,49 @@
         </gazebo>
     </xacro:macro>
+    <!-- <xacro:macro name="limo_gps" params="parent_prefix frame_prefix *joint_pose">
+        <link name='${frame_prefix}_link'>
+            <pose>0 0 0 0 0 0</pose>
+            <inertial>
+                <mass value="0.1"/>
+                <origin xyz="0.0 0 0" rpy="0 0 0"/>
+                <inertia
+                    ixx="1e-6" ixy="0" ixz="0"
+                    iyy="1e-6" iyz="0"
+                    izz="1e-6"
+                />
+            </inertial>
+            <visual name='gps_visual'>
+                <origin xyz="0 0 0" rpy="0 0 0"/>
+                <geometry>
+                    <box size="0.02 0.02 0.02"/>
+                </geometry>
+                <material name='gps_material'>
+                    <color rgba="0.75 0.75 0.75 1" />
+                </material>
+            </visual>
+            <collision name='gps_collision'>
+                <origin xyz="0 0 0" rpy="0 0 0"/>
+                <geometry>
+                    <box size="0.02 0.02 0.02"/>
+                </geometry>
+            </collision>
+        </link>
+        <joint type="fixed" name="gps_joint">
+            <xacro:insert_block name="joint_pose"/>
+            <child link="${frame_prefix}_link"/>
+            <parent link="${parent_prefix}"/>
+        </joint>
+        <gazebo reference="${frame_prefix}_link">
+            <sensor name="gps_sensor" type="gps">
+                <always_on>true</always_on>
+                <update_rate>10</update_rate>
+                <plugin name="gps_plugin" filename="libgazebo_ros_gps.so">
+                    <ros>
+                        <namespace>/gps</namespace>
+                        <remapping>~/out:=data</remapping>
+                    </ros>
+                </plugin>
+            </sensor>
+        </gazebo>
+    </xacro:macro> -->
 </robot>

File: limo_description/urdf/properties.xacro (robot description, xacro)
@@ -10,5 +10,5 @@
     <xacro:property name="wheelbase" value="0.2"/>
     <!-- <xacro:property name="track" value="0.14"/> -->
-    <xacro:property name="track" value="0.14"/>
+    <xacro:property name="track" value="0.13"/>
     <xacro:property name="wheel_vertical_offset" value="-0.100998" />
     <xacro:property name="base_mass" value="2.1557"/>
