Commit message: fix urdf and rviz view

File: limo_description/urdf/gazbo_control.xacro (robot description, xacro)
@@ -75,83 +75,63 @@
         </joint>
     </ros2_control>
-    <!-- Base Physics -->
+    <gazebo reference="base_footprint">
+            <mu1>10</mu1>
+            <mu2>10</mu2>
+            <kp>10000000.0</kp>
+            <kd>1.0</kd>
+            <minDepth>0.01</minDepth>
+            <fdir1>1 0 0</fdir1>
+            <maxContacts value="64"/>
+        </gazebo>
     <gazebo reference="base_link">
-        <minDepth>0.0002</minDepth>
-        <kp value="1000000.0"/>
-        <kd value="100.0"/>
-    </gazebo>
-    <!-- Fixed Steering Joint Names in Gazebo -->
-    <gazebo reference="left_steering_hinge">
-        <friction>
-            <ode>
-                <mu>10.0</mu>
-                <mu2>10.0</mu2>
-            </ode>
-        </friction>
-        <minDepth>0.0002</minDepth>
-        <kp value="1000000.0"/>
-        <kd value="100.0"/>
+            <mu1>10</mu1>
+            <mu2>10</mu2>
+            <kp>10000000.0</kp>
+            <kd>1.0</kd>
+            <minDepth>0.01</minDepth>
+            <fdir1>1 0 0</fdir1>
+            <maxContacts value="64"/>
+        </gazebo>
+    <gazebo reference="inertial_link">
+        <mu1>10</mu1>
+        <mu2>10</mu2>
+        <kp>10000000.0</kp>
+        <kd>1.0</kd>
+        <minDepth>0.01</minDepth>
+        <fdir1>1 0 0</fdir1>
         <maxContacts value="64"/>
     </gazebo>
-    <gazebo reference="right_steering_hinge">
-        <friction>
-            <ode>
-                <mu>10.0</mu>
-                <mu2>10.0</mu2>
-            </ode>
-        </friction>
-        <minDepth>0.0002</minDepth>
-        <kp value="1000000.0"/>
-        <kd value="100.0"/>
+    <gazebo reference="main_steering_link">
+        <mu1>10</mu1>
+        <mu2>10</mu2>
+        <kp>10000000.0</kp>
+        <kd>1.0</kd>
+        <minDepth>0.01</minDepth>
+        <fdir1>1 0 0</fdir1>
         <maxContacts value="64"/>
     </gazebo>
-    <!-- Wheels Physics -->
-    <gazebo reference="front_left_wheel">
-        <friction>
-            <ode>
-                <mu>10.0</mu>
-                <mu2>10.0</mu2>
-            </ode>
-        </friction>
-        <minDepth>0.0002</minDepth>
-        <kp value="1000000.0"/>
-        <kd value="100.0"/>
-        <maxContacts value="64"/>
+    <gazebo reference="front_left_wheel_link">
+        <mu1>0.5</mu1>
+        <mu2>0.5</mu2>
+        <kp>1000.0</kp>
+        <kd>1000.0</kd>
     </gazebo>
-    <gazebo reference="front_right_wheel">
-        <friction>
-            <ode>
-                <mu>10.0</mu>
-                <mu2>10.0</mu2>
-            </ode>
-        </friction>
-        <minDepth>0.0002</minDepth>
-        <kp value="1000000.0"/>
-        <kd value="100.0"/>
-        <maxContacts value="64"/>
+    <gazebo reference="front_right_wheel_link">
+        <mu1>0.5</mu1>
+        <mu2>0.5</mu2>
+        <kp>1000.0</kp>
+        <kd>1000.0</kd>
     </gazebo>
-    <gazebo reference="rear_left_wheel">
-        <friction>
-            <ode>
-                <mu>10.0</mu>
-                <mu2>10.0</mu2>
-            </ode>
-        </friction>
-        <minDepth>0.0002</minDepth>
-        <kp value="1000000.0"/>
-        <kd value="100.0"/>
-        <maxContacts value="64"/>
+    <gazebo reference="rear_left_wheel_link">
+        <mu1>0.5</mu1>
+        <mu2>0.5</mu2>
+        <kp>1000.0</kp>
+        <kd>1000.0</kd>
     </gazebo>
-    <gazebo reference="rear_right_wheel">
-        <friction>
-            <ode>
-                <mu>10.0</mu>
-                <mu2>10.0</mu2>
-            </ode>
-        </friction>
-        <minDepth>0.0002</minDepth>
-        <kp value="1000000.0"/>
-        <kd value="100.0"/>
-        <maxContacts value="64"/>
+    <gazebo reference="rear_right_wheel_link">
+        <mu1>0.5</mu1>
+        <mu2>0.5</mu2>
+        <kp>1000.0</kp>
+        <kd>1000.0</kd>
     </gazebo>
 </robot>

File: limo_description/urdf/limo_ackerman.xacro (robot description, xacro)
@@ -6,5 +6,5 @@
     <xacro:include filename="$(find limo_description)/urdf/inertial_macros.xacro" />
     <xacro:include filename="$(find limo_description)/urdf/properties.xacro" />
-    <xacro:include filename="$(find limo_description)/urdf/gazbo_control.xacro" />
+    <!-- <xacro:include filename="$(find limo_description)/urdf/gazbo_control.xacro" /> -->
     <link name="base_footprint"/>
     <joint name="base_joint" type="fixed">
@@ -13,10 +13,10 @@
         <origin xyz="0.0 0.0 0.15" rpy="0 0 0"/>
     </joint>
-    <!-- Base link -->
+        <!-- Base link -->
     <link name="base_link">
         <visual>
             <origin xyz="0 0 -0.15" rpy="0 0 1.57" />
             <geometry>
-                <mesh filename="file:///$(find limo_description)/meshes/limo_base.dae" scale="1 1 1"/>
+                <mesh filename="file://$(find limo_description)/meshes/limo_optimal.dae" scale="1 1 1"/>
             </geometry>
         </visual>
@@ -29,11 +29,11 @@
         <xacro:box_inertial_matrix  m="${base_mass}" w="${base_x_size}" l="${base_y_size}" h="${base_z_size}" />
     </link>
-    <link name="inertial_link">
+   <link name="inertial_link">
         <inertial>
             <origin xyz="0.0 0.0 0.0" />
             <mass value="${base_mass}" />
-            <inertia ixx="0.24" ixy="0" ixz="0"
-                     iyy="0.96" iyz="0"
-                     izz="0.96" />
+            <inertia ixx="0.0043832566666666675" ixy="0" ixz="0"
+                     iyy="0.004832360833333334" iyz="0"
+                     izz="0.005622784166666667" />
         </inertial>
     </link>
@@ -47,5 +47,5 @@
     </xacro:limo_laser>
     <xacro:limo_depth_camera parent_prefix="base_link" frame_prefix="depth_camera">
-        <origin xyz="0.084 0 0.03" rpy="0 0 0"/>
+        <origin xyz="0.084 0 0.026" rpy="0 0 0"/>
     </xacro:limo_depth_camera>
     <xacro:limo_imu parent_prefix="base_link" frame_prefix="imu">
@@ -53,12 +53,45 @@
     </xacro:limo_imu>
     <!-- Front Wheel -->
-    <xacro:limo_left_steering_hinge parent_prefix="base_link" wheel_prefix="left_steering_hinge">
+    <!-- <xacro:limo_left_steering_hinge parent_prefix="base_link" wheel_prefix="left_steering_hinge">
         <origin xyz="${wheelbase/2} ${track/2} ${wheel_vertical_offset}" rpy="0 0  0" />
     </xacro:limo_left_steering_hinge>
     <xacro:limo_right_steering_hinge parent_prefix="base_link" wheel_prefix="right_steering_hinge">
         <origin xyz="${wheelbase/2} ${-track/2} ${wheel_vertical_offset}" rpy="${M_PI} 0 0" />
+    </xacro:limo_right_steering_hinge> -->
+    <xacro:limo_left_steering_hinge parent_prefix="base_link" wheel_prefix="front_left">
+        <origin xyz="${wheelbase/2} ${track/2} ${wheel_vertical_offset}" rpy="0 0  0" />
+    </xacro:limo_left_steering_hinge>
+    <xacro:limo_right_steering_hinge parent_prefix="base_link" wheel_prefix="front_right">
+        <origin xyz="${wheelbase/2} ${-track/2} ${wheel_vertical_offset}" rpy="${M_PI} 0 0" />
     </xacro:limo_right_steering_hinge>
+    <link name="main_steering_link">
+        <inertial>
+            <mass value="0.25" />
+            <inertia ixx="0.00525" ixy="0" ixz="0" iyy="0.00035" iyz="0" izz="0.00525" />
+            <origin xyz="0 0 0" />
+        </inertial>
+        <visual>
+            <origin xyz="0 0 0" rpy="0 0 0" />
+            <geometry>
+                <mesh filename="file://$(find limo_description)/meshes/steering.dae" scale="1 1 1"/>
+            </geometry>
+        </visual>
+    </link>
+    <joint name="main_steering" type="revolute">
+        <parent link="base_link"/>
+        <child link="main_steering_link"/>
+        <origin xyz="${wheelbase/2} 0.0 ${wheel_vertical_offset * -2.0}" rpy="${M_PI} 0 0" />
+        <axis xyz="0 0 -1" />
+        <limit lower="-0.523598767" upper="0.523598767" effort="1000" velocity="10.0" />
+        <dynamics damping="0.0" friction="0.0"/>
+    </joint>
     <!-- Back Wheel -->
-    <link name="rear_left_wheel_link">
+    <xacro:limo_wheel parent_prefix="base_link" wheel_prefix="rear_left" reflect="1" fixed_on="false">
+        <origin xyz="${-wheelbase/2} ${track/2} ${wheel_vertical_offset}" rpy="0 0 0" />
+    </xacro:limo_wheel>
+    <xacro:limo_wheel parent_prefix="base_link" wheel_prefix="rear_right" reflect="-1" fixed_on="false">
+        <origin xyz="${-wheelbase/2} ${-track/2} ${wheel_vertical_offset}" rpy="${M_PI} 0 0" />
+    </xacro:limo_wheel>
+    <!-- <link name="rear_left_wheel_link">
         <inertial>
             <origin xyz="0 0 0" />
@@ -111,4 +144,4 @@
         <origin xyz="${-wheelbase/2} ${-track/2} ${wheel_vertical_offset}" rpy="${M_PI} 0 0" />
         <axis xyz="0 -1 0"/>
-    </joint>
+    </joint> -->
 </robot>

File: limo_description/urdf/limo_steering_hinge.xacro (robot description, xacro)
@@ -8,33 +8,21 @@
         <link name="${wheel_prefix}">
             <inertial>
-                <!-- diese Daten kommen aus das Internet -->
-                <mass value="0.25" />
-                <inertia ixx="0.00525" ixy="0" ixz="0" iyy="0.00035" iyz="0" izz="0.00525" />
-                <origin xyz="0 0 0" />
+              <mass value="0.25" />
+              <inertia ixx="0.00525" ixy="0" ixz="0" iyy="0.00035" iyz="0" izz="0.00525" />
+              <origin xyz="0 0 0" />
             </inertial>
             <visual>
                 <origin xyz="0 0 0" rpy="0 0 0" />
                 <geometry>
-                    <!-- es ist sehr klein -->
-                    <cylinder length="0.0001" radius="0.0001" />
+                  <cylinder length="0.0001" radius="0.0001" />
                 </geometry>
             </visual>
-            <collision>
-                <origin xyz="0 ${wheel_length/2} 0" rpy="1.57 0 0" />
-                <geometry>
-                    <cylinder length="${wheel_length}" radius="${wheel_radius-0.01}" />
-                </geometry>
-            </collision>
+            <!-- <collision>
+              <origin xyz="0 ${wheel_length/2} 0" rpy="1.57 0 0" />
+              <geometry>
+                  <cylinder length="${wheel_length}" radius="${wheel_radius-0.01}" />
+              </geometry>
+            </collision> -->
         </link>
-        <transmission name="${wheel_prefix}_hinge_trans" type="SimpleTransmission">
-            <type>transmission_interface/SimpleTransmission</type>
-            <actuator name="${wheel_prefix}_hinge_motor">
-                <hardwareInterface>hardware_interface/EffortJointInterface</hardwareInterface>
-                <mechanicalReduction>1</mechanicalReduction>
-            </actuator>
-            <joint name="${wheel_prefix}_steer_joint">
-                <hardwareInterface>hardware_interface/EffortJointInterface</hardwareInterface>
-            </joint>
-        </transmission>
         <joint name="${wheel_prefix}_steering" type="revolute">
             <parent link="${parent_prefix}"/>
@@ -42,53 +30,53 @@
             <xacro:insert_block name="joint_pose"/>
             <axis xyz="0 0 1" />
-            <limit lower="-0.523598767" upper="0.523598767" effort="5" velocity="0.5" />
-            <dynamics damping="1.0" friction="2.0"/>
+            <limit lower="-0.523598767" upper="0.523598767" effort="1000" velocity="1.0" />
+            <dynamics damping="0.0" friction="2.0"/>
         </joint>
-        <link name="front_left_wheel_link">
-            <inertial>
-                <mass value="0.25" />
-                <inertia ixx="0.00525" ixy="0" ixz="0" iyy="0.00035" iyz="0" izz="0.00525" />
-                <origin xyz="0 0 0" />
-            </inertial>
+        <link name="${wheel_prefix}_wheel_link">
+          <inertial>
+            <mass value="0.25" />
+            <inertia ixx="0.00525" ixy="0" ixz="0" iyy="0.00035" iyz="0" izz="0.00525" />
+            <origin xyz="0 0 0" />
+          </inertial>
+          <visual>
+              <origin xyz="0 0 0" rpy="0 0 0" />
+              <geometry>
+                  <mesh filename="file://$(find limo_description)/meshes/limo_optimal_wheels.dae" />
+              </geometry>
+          </visual>
+          <collision>
+            <origin xyz="0 ${wheel_length/2} 0" rpy="1.57 0 0" />
+            <geometry>
+                <cylinder length="${wheel_length}" radius="${wheel_radius}" />
+            </geometry>
+          </collision>
+      </link>
+        <joint name="${wheel_prefix}_wheel" type="continuous">
+          <parent link="${wheel_prefix}"/>
+          <child link="${wheel_prefix}_wheel_link"/>
+          <origin xyz="0 0 0" rpy="0 0  0" />
+          <axis xyz="0 1 0"/>
+          <limit effort="100.0" velocity="10.0"/>
+      </joint>
+    </xacro:macro>
+     <xacro:macro name="limo_right_steering_hinge" params="parent_prefix wheel_prefix *joint_pose">
+        <link name="${wheel_prefix}">
+          <inertial>
+            <mass value="0.25" />
+            <inertia ixx="0.00525" ixy="0" ixz="0" iyy="0.00035" iyz="0" izz="0.00525" />
+            <origin xyz="0 0 0" />
+          </inertial>
             <visual>
                 <origin xyz="0 0 0" rpy="0 0 0" />
                 <geometry>
-                    <mesh filename="file:///$(find limo_description)/meshes/limo_optimal_wheels.dae" />
+                  <cylinder length="0.0001" radius="0.0001" />
                 </geometry>
             </visual>
-            <collision>
-                <origin xyz="0 ${wheel_length/2} 0" rpy="1.57 0 0" />
-                <geometry>
-                    <cylinder length="${wheel_length}" radius="${wheel_radius}" />
-                </geometry>
-            </collision>
-            <xacro:cylinder_inertial_matrix  m="${wheel_mass}" r="${wheel_radius}"  h="${wheel_length}" />
-        </link>
-        <joint name="front_left_wheel" type="continuous">
-            <parent link="${wheel_prefix}"/>
-            <child link="front_left_wheel_link"/>
-            <origin xyz="0 0 0" rpy="0 0 0" />
-            <axis xyz="0 1 0"/>
-        </joint>
-    </xacro:macro>
-    <xacro:macro name="limo_right_steering_hinge" params="parent_prefix wheel_prefix *joint_pose">
-        <link name="${wheel_prefix}">
-            <inertial>
-                <mass value="0.25" />
-                <inertia ixx="0.00525" ixy="0" ixz="0" iyy="0.00035" iyz="0" izz="0.00525" />
-                <origin xyz="0 0 0" />
-            </inertial>
-            <visual>
-                <origin xyz="0 0 0" rpy="0 0 0" />
-                <geometry>
-                    <cylinder length="0.0001" radius="0.0001" />
-                </geometry>
-            </visual>
-            <collision>
+            <!-- <collision>
               <origin xyz="0 ${wheel_length/2} 0" rpy="1.57 0 0" />
               <geometry>
                   <cylinder length="${wheel_length}" radius="${wheel_radius-0.01}" />
               </geometry>
-            </collision>
+            </collision> -->
         </link>
         <joint name="${wheel_prefix}_steering" type="revolute">
@@ -97,33 +85,33 @@
             <xacro:insert_block name="joint_pose"/>
             <axis xyz="0 0 -1"/>
-            <limit lower="-0.6" upper="0.6" effort="20" velocity="2.0"/> <!-- Increased limits -->
-            <dynamics damping="1.0" friction="2.0"/>
+            <limit lower="-0.523598767" upper="0.523598767" effort="1000" velocity="1.0" />
+            <dynamics damping="0.0" friction="2.0"/>
         </joint>
         <link name="front_right_wheel_link">
-            <inertial>
-                <mass value="0.25" />
-                <inertia ixx="0.00525" ixy="0" ixz="0" iyy="0.00035" iyz="0" izz="0.00525" />
-                <origin xyz="0 0 0" />
-            </inertial>
-            <visual>
-                <origin xyz="0 0 0" rpy="0 0 0" />
-                <geometry>
-                    <mesh filename="file:///$(find limo_description)/meshes/limo_optimal_wheels.dae" />
-                </geometry>
-            </visual>
-            <collision>
-                <origin xyz="0 ${wheel_length/2} 0" rpy="1.57 0 0" />
-                <geometry>
-                    <cylinder length="${wheel_length}" radius="${wheel_radius}" />
-                </geometry>
-            </collision>
-            <xacro:cylinder_inertial_matrix  m="${wheel_mass}" r="${wheel_radius}"  h="${wheel_length}" />
-        </link>
-        <joint name="front_right_wheel" type="continuous">
-            <parent link="${wheel_prefix}"/>
-            <child link="front_right_wheel_link"/>
-            <origin xyz="0 0 0" rpy="0 0  0" />
-            <axis xyz="0 -1 0"/>
-        </joint>
+          <inertial>
+            <mass value="0.25" />
+            <inertia ixx="0.00525" ixy="0" ixz="0" iyy="0.00035" iyz="0" izz="0.00525" />
+            <origin xyz="0 0 0" />
+          </inertial>
+          <visual>
+              <origin xyz="0 0 0" rpy="0 0 0" />
+              <geometry>
+                  <mesh filename="file://$(find limo_description)/meshes/limo_optimal_wheels.dae" />
+              </geometry>
+          </visual>
+          <collision>
+            <origin xyz="0 ${wheel_length/2} 0" rpy="1.57 0 0" />
+            <geometry>
+                <cylinder length="${wheel_length}" radius="${wheel_radius}" />
+            </geometry>
+          </collision>
+      </link>
+      <joint name="${wheel_prefix}_wheel" type="continuous">
+          <parent link="${wheel_prefix}"/>
+          <child link="front_right_wheel_link"/>
+          <origin xyz="0 0 0" rpy="0 0  0" />
+          <axis xyz="0 -1 0"/>
+          <limit effort="100.0" velocity="10.0"/>
+      </joint>
     </xacro:macro>
 </robot>
