Commit message: fix urdf and rviz view

File: limo_description/urdf/limo_xacro.xacro (robot description, xacro)
@@ -1,17 +1,20 @@
 <?xml version="1.0"?>
 <robot name="limo_xacro" xmlns:xacro="http://ros.org/wiki/xacro">
-    <!-- <xacro:macro name="limo_wheel" params="parent_prefix wheel_prefix reflect *joint_pose">
+    <xacro:macro name="limo_wheel" params="parent_prefix wheel_prefix reflect *joint_pose visual_on:=true fixed_on:=false">
         <link name="${wheel_prefix}_wheel_link">
             <inertial>
-                <origin xyz="0 0 0" />
+                <origin xyz="0 ${wheel_length/2} 0" rpy="1.57 0 0" />
                 <mass value="0.5" />
-                <inertia ixx="0.01055" ixy="0" ixz="0" iyy="0.00075" iyz="0" izz="0.01055" />
+                <inertia ixx="0.00033749999999999996" ixy="0" ixz="0" iyy="0.00033749999999999996" iyz="0" izz="0.00050625" />
             </inertial>
-            <visual>
-                <origin xyz="0 0 0" rpy="0 0 0" />
-                <geometry>
-                    <mesh filename="file:///$(find limo_description)/meshes/limo_optimal_wheels.dae" />
-                </geometry>
-            </visual>
+            <xacro:if value="${visual_on}">
+                <visual>
+                    <origin xyz="0 0 0" rpy="0 0 0" />
+                    <geometry>
+                        <mesh filename="file://$(find limo_description)/meshes/limo_optimal_wheels.dae" />
+                        <!-- <mesh filename="file://$(find limo_description)/meshes/limo_optimal_wheels.dae" /> -->
+                    </geometry>
+                </visual>
+            </xacro:if>
             <collision>
               <origin xyz="0 ${wheel_length/2} 0" rpy="1.57 0 0" />
@@ -21,11 +24,22 @@
             </collision>
         </link>
-        <joint name="${wheel_prefix}_wheel" type="continuous">
-            <parent link="${parent_prefix}"/>
-            <child link="${wheel_prefix}_wheel_link"/>
-            <xacro:insert_block name="joint_pose"/>
-            <axis xyz="0 ${reflect*1} 0"/>
-        </joint>
-    </xacro:macro> -->
+        <!-- Conditionally set the joint type -->
+        <xacro:if value="${fixed_on}">
+            <joint name="${wheel_prefix}_wheel" type="fixed">
+                <parent link="${parent_prefix}"/>
+                <child link="${wheel_prefix}_wheel_link"/>
+                <xacro:insert_block name="joint_pose"/>
+            </joint>
+        </xacro:if>
+        <xacro:unless value="${fixed_on}">
+            <joint name="${wheel_prefix}_wheel" type="continuous">
+                <parent link="${parent_prefix}"/>
+                <child link="${wheel_prefix}_wheel_link"/>
+                <xacro:insert_block name="joint_pose"/>
+                <axis xyz="0 ${reflect*1} 0"/>
+                <limit effort="100.0" velocity="10.0"/>
+            </joint>
+        </xacro:unless>
+    </xacro:macro>
     <xacro:macro name="limo_laser" params="parent_prefix frame_prefix *joint_pose">
         <link name='${frame_prefix}_link'>
@@ -66,35 +80,35 @@
         <gazebo reference="${frame_prefix}_link">
             <material>Gazebo/Yellow</material>
-            <sensor type="ray" name="laser_sensor">
-              <pose>0 0 0 0 0 0</pose>
-              <visualize>false</visualize>
-              <update_rate>8</update_rate>
-              <ray>
+            <sensor name="laser" type="ray">
+            <always_on>true</always_on>
+            <visualize>false</visualize>
+            <update_rate>10</update_rate>
+            <ray>
                 <scan>
-                  <horizontal>
-                    <samples>720</samples>
-                    <resolution>1</resolution>
-                    <min_angle>-2.09439504</min_angle>
-                    <max_angle>2.09439504</max_angle>
-                  </horizontal>
+                <horizontal>
+                    <samples>120</samples>
+                    <resolution>1.000000</resolution>
+                    <min_angle>-3.14159</min_angle>
+                    <max_angle>3.14159</max_angle>
+                </horizontal>
                 </scan>
                 <range>
-                  <min>0.05</min>
-                  <max>8.0</max>
-                  <resolution>0.01</resolution>
+                <min>0.3</min>
+                <max>15.0</max>
+                <resolution>0.015</resolution>
                 </range>
                 <noise>
-                  <type>gaussian</type>
-                  <mean>0.0</mean>
-                  <stddev>0.01</stddev>
+                <type>gaussian</type>
+                <mean>0.0</mean>
+                <stddev>0.01</stddev>
                 </noise>
-              </ray>
-              <plugin name="gazebo_ros_laser_sensor" filename="libgazebo_ros_ray_sensor.so">
-              <ros>
+            </ray>
+            <plugin name="scan" filename="libgazebo_ros_ray_sensor.so">
+                <ros>
                 <remapping>~/out:=scan</remapping>
-              </ros>
-                <topicName>/limo/scan</topicName>
-                <frameName>laser_link</frameName>
-              </plugin>
+                </ros>
+                <output_type>sensor_msgs/LaserScan</output_type>
+                <frame_name>laser_link</frame_name>
+            </plugin>
             </sensor>
         </gazebo>
@@ -112,16 +126,10 @@
                 />
             </inertial>
-            <visual name='depth_camera_visual'>
+            <!-- <visual name='depth_camera_visual'>
                 <origin xyz="0 0 0" rpy="0 0 0"/>
                 <geometry>
                     <box size="0.02 0.06 0.015"/>
                 </geometry>
-                <material name='depth_camera_material'>
-                    <ambient>0.1 0.1 0.1 1</ambient>
-                    <diffuse>0.1 0.1 0.2 1</diffuse>
-                    <specular>0 0 0 0</specular>
-                    <emissive>0 0 0 1</emissive>
-                </material>
-            </visual>
+            </visual> -->
             <collision name='depth_camera_collision'>
                 <origin xyz="0 0 0" rpy="0 0 0"/>
@@ -141,50 +149,42 @@
             <parent link="${frame_prefix}_link"/>
             <child link="depth_link"/>
-          </joint>
+        </joint>
+            <link name="camera_depth_optical_frame"/>
+        <joint name="camera_depth_optical_joint" type="fixed">
+            <origin xyz="0 0 0" rpy="${-M_PI/2} 0 ${-M_PI/2}" />
+            <parent link="depth_camera_link" />
+            <child link="camera_depth_optical_frame" />
+        </joint>
         <gazebo reference="${frame_prefix}_link">
             <material>Gazebo/Yellow</material>
             <sensor name="sensor_camera" type="depth">
                 <pose>0.0 0.0 0.0 0.0 0.0 0.0</pose>
-                <always_on>true</always_on>
-                <visualize>true</visualize>
-                <update_rate>10.0</update_rate>
-                <camera name="head">
-                <horizontal_fov>1.3962634</horizontal_fov>
+                <always_on>1</always_on>
+                <update_rate>10</update_rate>
+                <visualize>1</visualize>
+                <camera name="limo_camera">
                 <image>
-                    <width>640</width>
-                    <height>480</height>
                     <format>R8G8B8</format>
+                    <width>400</width>
+                    <height>400</height>
                 </image>
                 <clip>
-                    <near>0.02</near>
-                    <far>300</far>
+                    <near>0.01</near>
+                    <far>10.0</far>
                 </clip>
                 </camera>
-                <plugin name="gazebo_ros_depth_camera_sensor" filename="libgazebo_ros_openni_kinect.so">
-                <baseline>0.2</baseline>
-                <alwaysOn>true</alwaysOn>
-                <!-- Keep this zero, update_rate in the parent <sensor> tag
-                    will control the frame rate. -->
-                <updateRate>0.0</updateRate>
-                <cameraName>camera_ir</cameraName>
-                <imageTopicName>/limo/color/image_raw</imageTopicName>
-                <cameraInfoTopicName>/limo/color/camera_info</cameraInfoTopicName>
-                <depthImageTopicName>/limo/depth/image_raw</depthImageTopicName>
-                <depthImageCameraInfoTopicName>/limo/depth/camera_info</depthImageCameraInfoTopicName>
-                <pointCloudTopicName>/limo/depth/points</pointCloudTopicName>
-                <frameName>depth_link</frameName>
-                <cameraname>depth_camera_link</cameraname>
-                <pointCloudCutoff>0.5</pointCloudCutoff>
-                <pointCloudCutoffMax>3.0</pointCloudCutoffMax>
-                <distortionK1>0</distortionK1>
-                <distortionK2>0</distortionK2>
-                <distortionK3>0</distortionK3>
-                <distortionT1>0</distortionT1>
-                <distortionT2>0</distortionT2>
-                <CxPrime>0</CxPrime>
-                <Cx>0</Cx>
-                <Cy>0</Cy>
-                <focalLength>0</focalLength>
-                <hackBaseline>0</hackBaseline>
+                <plugin name="gazebo_ros_depth_camera_sensor" filename="libgazebo_ros_camera.so">
+                <ros>
+                    <namespace>/limo</namespace>
+                    <argument>limo_camera/image_raw:=limo_camera/image</argument>
+                    <argument>limo_camera/image_depth:=limo_camera/depth/camera_image_depth</argument>
+                    <argument>limo_camera/camera_info:=limo_camera/camera_info_raw</argument>
+                    <argument>limo_camera/camera_info_depth:=limo_camera/camera_info_depth</argument>
+                    <argument>limo_camera/points:=limo_camera/camera_points</argument>
+                </ros>
+                <camera_name>depth_camera_link</camera_name>
+                <frame_name>camera_depth_optical_frame</frame_name>
+                <hack_baseline>0.07</hack_baseline>
+                <min_depth>0.001</min_depth>
                 </plugin>
             </sensor>
@@ -230,19 +230,77 @@
             <material>Gazebo/Yellow</material>
             <gravity>true</gravity>
-            <sensor name="imu_sensor" type="imu">
-                <always_on>true</always_on>
-                <update_rate>100</update_rate>
-                <visualize>true</visualize>
-                <topic>__default_topic__</topic>
-                <plugin filename="libgazebo_ros_imu_sensor.so" name="imu_plugin">
-                    <topicName>/limo/imu</topicName>
-                    <bodyName>${frame_prefix}_link</bodyName>
-                    <updateRateHZ>100.0</updateRateHZ>
-                    <gaussianNoise>0.001</gaussianNoise>
-                    <xyzOffset>0 0 0</xyzOffset>
-                    <rpyOffset>0 0 0</rpyOffset>
-                    <frameName>imu_link</frameName>
-                </plugin>
-                <pose>0 0 0 0 0 0</pose>
+            <sensor name="twr_imu" type="imu">
+            <always_on>true</always_on>
+            <update_rate>100</update_rate>
+            <visualize>true</visualize>
+            <imu>
+                <orientation>
+                <x>
+                    <noise type="gaussian">
+                    <mean>0.0</mean>
+                    <stddev>2e-3</stddev>
+                    </noise>
+                </x>
+                <y>
+                    <noise type="gaussian">
+                    <mean>0.0</mean>
+                    <stddev>2e-3</stddev>
+                    </noise>
+                </y>
+                <z>
+                    <noise type="gaussian">
+                    <mean>0.0</mean>
+                    <stddev>2e-3</stddev>
+                    </noise>
+                </z>
+                </orientation>
+                <angular_velocity>
+                <x>
+                    <noise type="gaussian">
+                    <mean>0.0</mean>
+                    <stddev>2e-4</stddev>
+                    </noise>
+                </x>
+                <y>
+                    <noise type="gaussian">
+                    <mean>0.0</mean>
+                    <stddev>2e-4</stddev>
+                    </noise>
+                </y>
+                <z>
+                    <noise type="gaussian">
+                    <mean>0.0</mean>
+                    <stddev>2e-4</stddev>
+                    </noise>
+                </z>
+                </angular_velocity>
+                <linear_acceleration>
+                <x>
+                    <noise type="gaussian">
+                    <mean>0.0</mean>
+                    <stddev>1.7e-2</stddev>
+                    </noise>
+                </x>
+                <y>
+                    <noise type="gaussian">
+                    <mean>0.0</mean>
+                    <stddev>1.7e-2</stddev>
+                    </noise>
+                </y>
+                <z>
+                    <noise type="gaussian">
+                    <mean>0.0</mean>
+                    <stddev>1.7e-2</stddev>
+                    </noise>
+                </z>
+                </linear_acceleration>
+            </imu>
+            <plugin name="two_wheeled_robot_imu" filename="libgazebo_ros_imu_sensor.so">
+                <initial_orientation_as_reference>false</initial_orientation_as_reference>
+                <frame_name>imu_link</frame_name>
+                <ros>
+                <remapping>~/out:=imu</remapping>
+                </ros>
+            </plugin>
             </sensor>
         </gazebo>

File: limo_description/urdf/properties.xacro (robot description, xacro)
@@ -6,11 +6,11 @@
     <xacro:property name="base_x_size" value="0.13" />
     <xacro:property name="base_y_size" value="0.12" />
-    <xacro:property name="base_z_size" value="0.10" />
+    <xacro:property name="base_z_size" value="0.1" />
     <xacro:property name="wheelbase" value="0.2"/>
-    <xacro:property name="track" value="0.14"/>
-    <xacro:property name="wheel_vertical_offset" value="-0.100998" />
+    <xacro:property name="track" value="0.13"/>
+    <xacro:property name="wheel_vertical_offset" value="-0.10" />
     <xacro:property name="base_mass" value="2.1557"/>
     <xacro:property name="wheel_mass" value="0.5" />
-    <xacro:property name="wheel_length" value="0.045" />
+    <xacro:property name="wheel_length" value="0.001" />
     <xacro:property name="wheel_radius" value="0.045" />
 </robot>

Commit message: update gazebo launch file

File: limo_description/urdf/gazbo_control.xacro (robot description, xacro)
@@ -1,4 +1,4 @@
 <?xml version="1.0"?>
-<robot xmlns:xacro="http://www.ros.org/wiki/xacro" name="otto">
+<robot xmlns:xacro="http://www.ros.org/wiki/xacro">
     <gazebo>
         <plugin filename="libgazebo_ros2_control.so" name="gazebo_ros2_control">
@@ -10,37 +10,16 @@
             <plugin>gazebo_ros2_control/GazeboSystem</plugin>
         </hardware>
-        <!-- Steering Joints (Position Control) -->
-        <joint name="left_steering_hinge">
-            <command_interface name="position">
-                <param name="min">-0.6</param> <!-- Increased Steering Angle -->
-                <param name="max">0.6</param>
-            </command_interface>
-            <state_interface name="position"/>
-            <state_interface name="velocity"/>
-            <state_interface name="effort"/>
-            <limit effort="5" velocity="0.5"/> <!-- Added Limits -->
-            <axis xyz="0 0 1"/> <!-- Ensures Correct Steering Rotation -->
-        </joint>
-        <joint name="right_steering_hinge">
-            <command_interface name="position">
-                <param name="min">-0.6</param>
-                <param name="max">0.6</param>
-            </command_interface>
-            <state_interface name="position"/>
-            <state_interface name="velocity"/>
-            <state_interface name="effort"/>
-            <limit effort="5" velocity="0.5"/>
-            <axis xyz="0 0 1"/> <!-- Ensures Correct Steering Rotation -->
-        </joint>
-        <!-- Wheel Joints (Velocity Control) -->
         <joint name="front_left_wheel">
             <command_interface name="velocity">
                 <param name="min">-5</param>
                 <param name="max">5</param>
-            </command_interface>
-            <state_interface name="position"/>
-            <state_interface name="velocity"/>
-            <state_interface name="effort"/>
-            <limit effort="20" velocity="5"/> <!-- Added Limits -->
+              </command_interface>
+              <state_interface name="position">
+                <param name="initial_value">0.0</param>
+              </state_interface>
+              <state_interface name="velocity">
+                <param name="initial_value">0.0</param>
+              </state_interface>
+              <state_interface name="effort"/>
         </joint>
         <joint name="front_right_wheel">
@@ -48,9 +27,12 @@
                 <param name="min">-5</param>
                 <param name="max">5</param>
-            </command_interface>
-            <state_interface name="position"/>
-            <state_interface name="velocity"/>
-            <state_interface name="effort"/>
-            <limit effort="20" velocity="5"/>
+              </command_interface>
+              <state_interface name="position">
+                <param name="initial_value">0.0</param>
+              </state_interface>
+              <state_interface name="velocity">
+                <param name="initial_value">0.0</param>
+              </state_interface>
+              <state_interface name="effort"/>
         </joint>
         <joint name="rear_left_wheel">
@@ -58,9 +40,12 @@
                 <param name="min">-5</param>
                 <param name="max">5</param>
-            </command_interface>
-            <state_interface name="position"/>
-            <state_interface name="velocity"/>
-            <state_interface name="effort"/>
-            <limit effort="20" velocity="5"/>
+              </command_interface>
+              <state_interface name="position">
+                <param name="initial_value">0.0</param>
+              </state_interface>
+              <state_interface name="velocity">
+                <param name="initial_value">0.0</param>
+              </state_interface>
+              <state_interface name="effort"/>
         </joint>
         <joint name="rear_right_wheel">
@@ -68,9 +53,51 @@
                 <param name="min">-5</param>
                 <param name="max">5</param>
-            </command_interface>
-            <state_interface name="position"/>
-            <state_interface name="velocity"/>
-            <state_interface name="effort"/>
-            <limit effort="20" velocity="5"/>
+              </command_interface>
+              <state_interface name="position">
+                <param name="initial_value">0.0</param>
+              </state_interface>
+              <state_interface name="velocity">
+                <param name="initial_value">0.0</param>
+              </state_interface>
+              <state_interface name="effort"/>
+        </joint>
+        <joint name="main_steering">
+            <command_interface name="position">
+                <param name="min">-0.523598767</param>
+                <param name="max">0.523598767</param>
+              </command_interface>
+              <state_interface name="position">
+                <param name="initial_value">0.0</param>
+              </state_interface>
+              <state_interface name="velocity">
+                <param name="initial_value">0.0</param>
+              </state_interface>
+              <state_interface name="effort"/>
+        </joint>
+        <joint name="front_left_steering">
+            <command_interface name="velocity"/>
+            <command_interface name="position">
+                <param name="min">-0.523598767</param>
+                <param name="max">0.523598767</param>
+              </command_interface>
+              <state_interface name="position">
+                <param name="initial_value">0.0</param>
+              </state_interface>
+              <state_interface name="velocity">
+              </state_interface>
+              <state_interface name="effort"/>
+        </joint>
+        <joint name="front_right_steering">
+            <command_interface name="velocity"/>
+            <command_interface name="position">
+                <param name="min">-0.523598767</param>
+                <param name="max">0.523598767</param>
+              </command_interface>
+              <state_interface name="position">
+                <param name="initial_value">0.0</param>
+              </state_interface>
+              <state_interface name="velocity">
+              </state_interface>
+              <state_interface name="effort"/>
         </joint>
     </ros2_control>

File: limo_description/urdf/limo_ackerman.xacro (robot description, xacro)
@@ -6,5 +6,5 @@
     <xacro:include filename="$(find limo_description)/urdf/inertial_macros.xacro" />
     <xacro:include filename="$(find limo_description)/urdf/properties.xacro" />
-    <!-- <xacro:include filename="$(find limo_description)/urdf/gazbo_control.xacro" /> -->
+    <xacro:include filename="$(find limo_description)/urdf/gazbo_control.xacro" />
     <link name="base_footprint"/>
     <joint name="base_joint" type="fixed">
