Commit message: add test simple controller

File: limo_description/urdf/gazbo_control.xacro (robot description, xacro)
@@ -12,6 +12,6 @@
         <joint name="front_left_wheel">
             <command_interface name="velocity">
-                <param name="min">-5</param>
-                <param name="max">5</param>
+                <param name="min">-10</param>
+                <param name="max">10</param>
               </command_interface>
               <state_interface name="position">
@@ -25,6 +25,6 @@
         <joint name="front_right_wheel">
             <command_interface name="velocity">
-                <param name="min">-5</param>
-                <param name="max">5</param>
+                <param name="min">-10</param>
+                <param name="max">10</param>
               </command_interface>
               <state_interface name="position">
@@ -38,6 +38,6 @@
         <joint name="rear_left_wheel">
             <command_interface name="velocity">
-                <param name="min">-5</param>
-                <param name="max">5</param>
+                <param name="min">-10</param>
+                <param name="max">10</param>
               </command_interface>
               <state_interface name="position">
@@ -51,19 +51,6 @@
         <joint name="rear_right_wheel">
             <command_interface name="velocity">
-                <param name="min">-5</param>
-                <param name="max">5</param>
-              </command_interface>
-              <state_interface name="position">
-                <param name="initial_value">0.0</param>
-              </state_interface>
-              <state_interface name="velocity">
-                <param name="initial_value">0.0</param>
-              </state_interface>
-              <state_interface name="effort"/>
-        </joint>
-        <joint name="main_steering">
-            <command_interface name="position">
-                <param name="min">-0.523598767</param>
-                <param name="max">0.523598767</param>
+                <param name="min">-10</param>
+                <param name="max">10</param>
               </command_interface>
               <state_interface name="position">
@@ -120,45 +107,31 @@
             <maxContacts value="64"/>
         </gazebo>
-    <gazebo reference="inertial_link">
-        <mu1>10</mu1>
-        <mu2>10</mu2>
-        <kp>10000000.0</kp>
-        <kd>1.0</kd>
-        <minDepth>0.01</minDepth>
-        <fdir1>1 0 0</fdir1>
-        <maxContacts value="64"/>
-    </gazebo>
-    <gazebo reference="main_steering_link">
-        <mu1>10</mu1>
-        <mu2>10</mu2>
-        <kp>10000000.0</kp>
-        <kd>1.0</kd>
-        <minDepth>0.01</minDepth>
-        <fdir1>1 0 0</fdir1>
-        <maxContacts value="64"/>
-    </gazebo>
     <gazebo reference="front_left_wheel_link">
-        <mu1>0.5</mu1>
-        <mu2>0.5</mu2>
-        <kp>1000.0</kp>
-        <kd>1000.0</kd>
+        <mu1>10.0</mu1>
+        <mu2>10.0</mu2>
+        <minDepth>0.0002</minDepth>
+        <kp  value="1000000.0"/>
+        <kd  value="100.0"/>
     </gazebo>
     <gazebo reference="front_right_wheel_link">
-        <mu1>0.5</mu1>
-        <mu2>0.5</mu2>
-        <kp>1000.0</kp>
-        <kd>1000.0</kd>
+        <mu1>10.0</mu1>
+        <mu2>10.0</mu2>
+        <minDepth>0.0002</minDepth>
+        <kp  value="1000000.0"/>
+        <kd  value="100.0"/>
     </gazebo>
     <gazebo reference="rear_left_wheel_link">
-        <mu1>0.5</mu1>
-        <mu2>0.5</mu2>
-        <kp>1000.0</kp>
-        <kd>1000.0</kd>
+        <mu1>10.0</mu1>
+        <mu2>10.0</mu2>
+        <minDepth>0.0002</minDepth>
+        <kp  value="1000000.0"/>
+        <kd  value="100.0"/>
     </gazebo>
     <gazebo reference="rear_right_wheel_link">
-        <mu1>0.5</mu1>
-        <mu2>0.5</mu2>
-        <kp>1000.0</kp>
-        <kd>1000.0</kd>
+        <mu1>10.0</mu1>
+        <mu2>10.0</mu2>
+        <minDepth>0.0002</minDepth>
+        <kp  value="1000000.0"/>
+        <kd  value="100.0"/>
     </gazebo>
 </robot>

File: limo_description/urdf/inertial_macros.xacro (robot description, xacro)
@@ -1,4 +1,14 @@
 <?xml version="1.0"?>
 <robot xmlns:xacro="http://ros.org/wiki/xacro">
+    <xacro:macro name="sphere_inertial_matrix" params="m r">
+        <inertial>
+            <origin xyz="0.0 0.0 0.0" />
+            <mass value="${m}" />
+            <inertia ixx="${2*m*r*r/5}" ixy="0" ixz="0"
+                     iyy="${2*m*r*r/5}" iyz="0"
+                     izz="${2*m*r*r/5}" />
+        </inertial>
+    </xacro:macro>
+    <!-- Zylinder -->
     <xacro:macro name="cylinder_inertial_matrix" params="m r h">
         <inertial>

File: limo_description/urdf/limo_steering_hinge.xacro (robot description, xacro)
@@ -1,6 +1,3 @@
 <?xml version="1.0"?>
-<!--Auto: Zhui Li-->
-<!-- Description: Diese xacro-Datei basiert auf den Regeln und definiert Funktionen durch xacro,
-um die Erstellung von Steuerscharnier des Wagens zu ermöglichen. Durch Macrofunktion dient es einfach beim Aufruf in limo_base.-->
 <robot name="limo_steering_hinge" xmlns:xacro="http://www.ros.org/wiki/xacro">
     <xacro:include filename="$(find limo_description)/urdf/inertial_macros.xacro" />
@@ -18,10 +15,10 @@
                 </geometry>
             </visual>
-            <!-- <collision>
-              <origin xyz="0 ${wheel_length/2} 0" rpy="1.57 0 0" />
-              <geometry>
-                  <cylinder length="${wheel_length}" radius="${wheel_radius-0.01}" />
-              </geometry>
-            </collision> -->
+            <collision>
+                <origin xyz="0 ${wheel_length/2} 0" rpy="1.57 0 0" />
+                <geometry>
+                    <cylinder length="${wheel_length}" radius="${wheel_radius-0.01}" />
+                </geometry>
+            </collision>
         </link>
         <joint name="${wheel_prefix}_steering" type="revolute">
@@ -31,12 +28,12 @@
             <axis xyz="0 0 1" />
             <limit lower="-0.523598767" upper="0.523598767" effort="1000" velocity="1.0" />
-            <dynamics damping="0.0" friction="2.0"/>
+            <dynamics damping="1.0" friction="2.0"/>
         </joint>
         <link name="${wheel_prefix}_wheel_link">
-          <inertial>
+          <!-- <inertial>
             <mass value="0.25" />
             <inertia ixx="0.00525" ixy="0" ixz="0" iyy="0.00035" iyz="0" izz="0.00525" />
             <origin xyz="0 0 0" />
-          </inertial>
+          </inertial> -->
           <visual>
               <origin xyz="0 0 0" rpy="0 0 0" />
@@ -45,10 +42,11 @@
               </geometry>
           </visual>
-          <collision>
-            <origin xyz="0 ${wheel_length/2} 0" rpy="1.57 0 0" />
-            <geometry>
-                <cylinder length="${wheel_length}" radius="${wheel_radius}" />
-            </geometry>
-          </collision>
+            <collision>
+                <origin xyz="0 ${wheel_length/2} 0" rpy="1.57 0 0" />
+                <geometry>
+                    <cylinder length="${wheel_length}" radius="${wheel_radius}" />
+                </geometry>
+            </collision>
+            <xacro:cylinder_inertial_matrix  m="${wheel_mass}" r="${wheel_radius}"  h="${wheel_length}" />
       </link>
         <joint name="${wheel_prefix}_wheel" type="continuous">
@@ -73,10 +71,10 @@
                 </geometry>
             </visual>
-            <!-- <collision>
-              <origin xyz="0 ${wheel_length/2} 0" rpy="1.57 0 0" />
-              <geometry>
-                  <cylinder length="${wheel_length}" radius="${wheel_radius-0.01}" />
-              </geometry>
-            </collision> -->
+            <collision>
+                <origin xyz="0 ${wheel_length/2} 0" rpy="1.57 0 0" />
+                <geometry>
+                    <cylinder length="${wheel_length}" radius="${wheel_radius-0.01}" />
+                </geometry>
+            </collision>
         </link>
         <joint name="${wheel_prefix}_steering" type="revolute">
@@ -86,12 +84,12 @@
             <axis xyz="0 0 -1"/>
             <limit lower="-0.523598767" upper="0.523598767" effort="1000" velocity="1.0" />
-            <dynamics damping="0.0" friction="2.0"/>
+            <dynamics damping="1.0" friction="2.0"/>
         </joint>
         <link name="front_right_wheel_link">
-          <inertial>
+          <!-- <inertial>
             <mass value="0.25" />
             <inertia ixx="0.00525" ixy="0" ixz="0" iyy="0.00035" iyz="0" izz="0.00525" />
             <origin xyz="0 0 0" />
-          </inertial>
+          </inertial> -->
           <visual>
               <origin xyz="0 0 0" rpy="0 0 0" />
@@ -106,4 +104,5 @@
             </geometry>
           </collision>
+          <xacro:cylinder_inertial_matrix  m="${wheel_mass}" r="${wheel_radius}"  h="${wheel_length}" />
       </link>
       <joint name="${wheel_prefix}_wheel" type="continuous">

File: limo_description/urdf/limo_xacro.xacro (robot description, xacro)
@@ -1,11 +1,5 @@
 <?xml version="1.0"?>
 <robot name="limo_xacro" xmlns:xacro="http://ros.org/wiki/xacro">
-    <material name="laser_material">
-        <color rgba="1.0 1.0 0.0 1.0"/> <!-- Yellow -->
-    </material>
-    <material name="imu_material">
-        <color rgba="0.0 1.0 1.0 1.0"/> <!-- Cyan -->
-    </material>
-    <xacro:macro name="limo_wheel" params="parent_prefix wheel_prefix reflect *joint_pose visual_on:=true fixed_on:=false">
+    <!-- <xacro:macro name="limo_wheel" params="parent_prefix wheel_prefix reflect *joint_pose visual_on:=true fixed_on:=false">
         <link name="${wheel_prefix}_wheel_link">
             <inertial>
@@ -19,5 +13,4 @@
                     <geometry>
                         <mesh filename="file://$(find limo_description)/meshes/limo_optimal_wheels.dae" />
-                        <!-- <mesh filename="file://$(find limo_description)/meshes/limo_optimal_wheels.dae" /> -->
                     </geometry>
                 </visual>
@@ -29,7 +22,7 @@
               </geometry>
             </collision>
-        </link>
+        </link> -->
         <!-- Conditionally set the joint type -->
-        <xacro:if value="${fixed_on}">
+        <!-- <xacro:if value="${fixed_on}">
             <joint name="${wheel_prefix}_wheel" type="fixed">
                 <parent link="${parent_prefix}"/>
@@ -47,4 +40,32 @@
             </joint>
         </xacro:unless>
+    </xacro:macro> -->
+    <xacro:macro name="limo_wheel" params="parent_prefix wheel_prefix reflect *joint_pose">
+        <link name="${wheel_prefix}_wheel_link">
+            <!-- <inertial>
+                <origin xyz="0 0 0" />
+                <mass value="0.5" />
+                <inertia ixx="0.01055" ixy="0" ixz="0" iyy="0.00075" iyz="0" izz="0.01055" />
+            </inertial> -->
+            <visual>
+                <origin xyz="0 0 0" rpy="0 0 0" />
+                <geometry>
+                    <mesh filename="file://$(find limo_description)/meshes/limo_optimal_wheels.dae" />
+                </geometry>
+            </visual>
+            <collision>
+              <origin xyz="0 ${wheel_length/2} 0" rpy="1.57 0 0" />
+              <geometry>
+                  <cylinder length="${wheel_length}" radius="${wheel_radius}" />
+              </geometry>
+            </collision>
+            <xacro:cylinder_inertial_matrix  m="${wheel_mass}" r="${wheel_radius}"  h="${wheel_length}" />
+        </link>
+        <joint name="${wheel_prefix}_wheel" type="continuous">
+            <parent link="${parent_prefix}"/>
+            <child link="${wheel_prefix}_wheel_link"/>
+            <xacro:insert_block name="joint_pose"/>
+            <axis xyz="0 ${reflect*1} 0"/>
+        </joint>
     </xacro:macro>
     <xacro:macro name="limo_laser" params="parent_prefix frame_prefix *joint_pose">
@@ -66,4 +87,5 @@
                 </geometry>
                 <material name='laser_material'>
+                    <color rgba="0.75 0.75 0.75 1" />
                     <ambient>0.1 0.1 0.1 1</ambient>
                     <diffuse>0.1 0.1 0.2 1</diffuse>
@@ -217,4 +239,5 @@
                 </geometry>
                 <material name='imu_material'>
+                    <color rgba="0.75 0.75 0.75 1" />
                     <ambient>0.1 0.1 0.1 1</ambient>
                     <diffuse>0.1 0.1 0.2 1</diffuse>

File: limo_description/urdf/properties.xacro (robot description, xacro)
@@ -6,11 +6,11 @@
     <xacro:property name="base_x_size" value="0.13" />
     <xacro:property name="base_y_size" value="0.12" />
-    <xacro:property name="base_z_size" value="0.1" />
+    <xacro:property name="base_z_size" value="0.10" />
     <xacro:property name="wheelbase" value="0.2"/>
-    <xacro:property name="track" value="0.13"/>
-    <xacro:property name="wheel_vertical_offset" value="-0.10" />
+    <xacro:property name="track" value="0.14"/>
+    <xacro:property name="wheel_vertical_offset" value="-0.100998" />
     <xacro:property name="base_mass" value="2.1557"/>
     <xacro:property name="wheel_mass" value="0.5" />
-    <xacro:property name="wheel_length" value="0.001" />
+    <xacro:property name="wheel_length" value="0.045" />
     <xacro:property name="wheel_radius" value="0.045" />
 </robot>

Commit message: add ackermann controller

File: limo_description/urdf/gazbo_control.xacro (robot description, xacro)
@@ -90,21 +90,13 @@
     </ros2_control>
     <gazebo reference="base_footprint">
-            <mu1>10</mu1>
-            <mu2>10</mu2>
-            <kp>10000000.0</kp>
-            <kd>1.0</kd>
-            <minDepth>0.01</minDepth>
-            <fdir1>1 0 0</fdir1>
-            <maxContacts value="64"/>
-        </gazebo>
+        <minDepth>0.0002</minDepth>
+        <kp  value="1000000.0"/>
+        <kd  value="100.0"/>
+    </gazebo>
     <gazebo reference="base_link">
-            <mu1>10</mu1>
-            <mu2>10</mu2>
-            <kp>10000000.0</kp>
-            <kd>1.0</kd>
-            <minDepth>0.01</minDepth>
-            <fdir1>1 0 0</fdir1>
-            <maxContacts value="64"/>
-        </gazebo>
+        <minDepth>0.0002</minDepth>
+        <kp  value="1000000.0"/>
+        <kd  value="100.0"/>
+    </gazebo>
     <gazebo reference="front_left_wheel_link">
         <mu1>10.0</mu1>

File: limo_description/urdf/limo_steering_hinge.xacro (robot description, xacro)
@@ -28,5 +28,5 @@
             <axis xyz="0 0 1" />
             <limit lower="-0.523598767" upper="0.523598767" effort="1000" velocity="1.0" />
-            <dynamics damping="1.0" friction="2.0"/>
+            <dynamics damping="0.0" friction="2.0"/>
         </joint>
         <link name="${wheel_prefix}_wheel_link">
@@ -84,5 +84,5 @@
             <axis xyz="0 0 -1"/>
             <limit lower="-0.523598767" upper="0.523598767" effort="1000" velocity="1.0" />
-            <dynamics damping="1.0" friction="2.0"/>
+            <dynamics damping="0.0" friction="2.0"/>
         </joint>
         <link name="front_right_wheel_link">

Commit message: add last ackermann controller implement

File: limo_description/urdf/gazbo_control.xacro (robot description, xacro)
@@ -25,6 +25,6 @@
         <joint name="front_right_wheel">
             <command_interface name="velocity">
-                <param name="min">-10</param>
-                <param name="max">10</param>
+                <param name="min">-20</param>
+                <param name="max">20</param>
               </command_interface>
               <state_interface name="position">
@@ -38,6 +38,6 @@
         <joint name="rear_left_wheel">
             <command_interface name="velocity">
-                <param name="min">-10</param>
-                <param name="max">10</param>
+                <param name="min">-20</param>
+                <param name="max">20</param>
               </command_interface>
               <state_interface name="position">
@@ -51,6 +51,6 @@
         <joint name="rear_right_wheel">
             <command_interface name="velocity">
-                <param name="min">-10</param>
-                <param name="max">10</param>
+                <param name="min">-20</param>
+                <param name="max">20</param>
               </command_interface>
               <state_interface name="position">
@@ -88,4 +88,18 @@
               <state_interface name="effort"/>
         </joint>
+<!--
+        <joint name="main_steering">
+            <command_interface name="velocity"/>
+            <command_interface name="position">
+                <param name="min">-0.523598767</param>
+                <param name="max">0.523598767</param>
+              </command_interface>
+              <state_interface name="position">
+                <param name="initial_value">0.0</param>
+              </state_interface>
+              <state_interface name="velocity">
+              </state_interface>
+              <state_interface name="effort"/>
+        </joint> -->
     </ros2_control>
     <gazebo reference="base_footprint">
@@ -99,4 +113,10 @@
         <kd  value="100.0"/>
     </gazebo>
+<!--
+    <gazebo reference="main_steering_link">
+        <minDepth>0.0002</minDepth>
+        <kp  value="1000000.0"/>
+        <kd  value="100.0"/>
+    </gazebo> -->
     <gazebo reference="front_left_wheel_link">
         <mu1>10.0</mu1>

File: limo_description/urdf/limo_ackerman.urdf.xacro (robot description, xacro)
@@ -60,4 +60,25 @@
         <origin xyz="${wheelbase/2} ${-track/2} ${wheel_vertical_offset}" rpy="${M_PI} 0 0" />
     </xacro:limo_right_steering_hinge>
+    <!-- <link name="main_steering_link">
+        <inertial>
+            <mass value="0.25" />
+            <inertia ixx="0.00525" ixy="0" ixz="0" iyy="0.00035" iyz="0" izz="0.00525" />
+            <origin xyz="0 0 0" />
+        </inertial>
+        <visual>
+            <origin xyz="0 0 0" rpy="0 0 0" />
+            <geometry>
+                <mesh filename="file://$(find limo_description)/meshes/steering.dae" scale="1 1 1"/>
+            </geometry>
+        </visual>
+    </link>
+    <joint name="main_steering" type="revolute">
+        <parent link="base_link"/>
+        <child link="main_steering_link"/>
+        <origin xyz="${wheelbase/2} 0.0 ${wheel_vertical_offset * -2.0}" rpy="${M_PI} 0 0" />
+        <axis xyz="0 0 -1" />
+        <limit lower="-0.523598767" upper="0.523598767" effort="1000" velocity="10.0" />
+        <dynamics damping="0.0" friction="0.0"/>
+    </joint> -->
     <!-- Back Wheel -->
     <xacro:limo_wheel parent_prefix="base_link" wheel_prefix="rear_left" reflect="1" >

File: limo_description/urdf/limo_steering_hinge.xacro (robot description, xacro)
@@ -55,5 +55,5 @@
           <origin xyz="0 0 0" rpy="0 0  0" />
           <axis xyz="0 1 0"/>
-          <limit effort="100.0" velocity="10.0"/>
+          <!-- <limit effort="100.0" velocity="10.0"/> -->
       </joint>
     </xacro:macro>
@@ -111,5 +111,5 @@
           <origin xyz="0 0 0" rpy="0 0  0" />
           <axis xyz="0 -1 0"/>
-          <limit effort="100.0" velocity="10.0"/>
+          <!-- <limit effort="100.0" velocity="10.0"/> -->
       </joint>
     </xacro:macro>

File: limo_description/urdf/properties.xacro (robot description, xacro)
@@ -6,11 +6,14 @@
     <xacro:property name="base_x_size" value="0.13" />
     <xacro:property name="base_y_size" value="0.12" />
+    <!-- <xacro:property name="base_z_size" value="0.10" /> -->
     <xacro:property name="base_z_size" value="0.10" />
     <xacro:property name="wheelbase" value="0.2"/>
+    <!-- <xacro:property name="track" value="0.14"/> -->
     <xacro:property name="track" value="0.14"/>
     <xacro:property name="wheel_vertical_offset" value="-0.100998" />
     <xacro:property name="base_mass" value="2.1557"/>
     <xacro:property name="wheel_mass" value="0.5" />
-    <xacro:property name="wheel_length" value="0.045" />
+    <!-- <xacro:property name="wheel_length" value="0.045" /> -->
+    <xacro:property name="wheel_length" value="0.001" />
     <xacro:property name="wheel_radius" value="0.045" />
 </robot>
