Commit message: update noslip controller and yawrate odom

File: limo_description/urdf/gazbo_control.xacro (robot description, xacro)
@@ -25,6 +25,6 @@
         <joint name="front_right_wheel">
             <command_interface name="velocity">
-                <param name="min">-20</param>
-                <param name="max">20</param>
+                <param name="min">-10</param>
+                <param name="max">10</param>
               </command_interface>
               <state_interface name="position">
@@ -38,6 +38,6 @@
         <joint name="rear_left_wheel">
             <command_interface name="velocity">
-                <param name="min">-20</param>
-                <param name="max">20</param>
+                <param name="min">-10</param>
+                <param name="max">10</param>
               </command_interface>
               <state_interface name="position">
@@ -51,6 +51,6 @@
         <joint name="rear_right_wheel">
             <command_interface name="velocity">
-                <param name="min">-20</param>
-                <param name="max">20</param>
+                <param name="min">-10</param>
+                <param name="max">10</param>
               </command_interface>
               <state_interface name="position">
@@ -65,6 +65,6 @@
             <command_interface name="velocity"/>
             <command_interface name="position">
-                <param name="min">-0.523598767</param>
-                <param name="max">0.523598767</param>
+                <param name="min">-0.698132</param>
+                <param name="max">0.698132</param>
               </command_interface>
               <state_interface name="position">
@@ -78,6 +78,6 @@
             <command_interface name="velocity"/>
             <command_interface name="position">
-                <param name="min">-0.523598767</param>
-                <param name="max">0.523598767</param>
+                <param name="min">-0.698132</param>
+                <param name="max">0.698132</param>
               </command_interface>
               <state_interface name="position">

File: limo_description/urdf/limo_steering_hinge.xacro (robot description, xacro)
@@ -27,6 +27,6 @@
             <xacro:insert_block name="joint_pose"/>
             <axis xyz="0 0 1" />
-            <limit lower="-0.523598767" upper="0.523598767" effort="1000" velocity="1.0" />
-            <dynamics damping="0.0" friction="2.0"/>
+            <limit lower="-0.698132" upper="0.698132" effort="1000" velocity="1.0" />
+            <dynamics damping="1.0" friction="2.0"/>
         </joint>
         <link name="${wheel_prefix}_wheel_link">
@@ -55,5 +55,5 @@
           <origin xyz="0 0 0" rpy="0 0  0" />
           <axis xyz="0 1 0"/>
-          <!-- <limit effort="100.0" velocity="10.0"/> -->
+          <limit effort="100.0" velocity="10.0"/>
       </joint>
     </xacro:macro>
@@ -83,6 +83,6 @@
             <xacro:insert_block name="joint_pose"/>
             <axis xyz="0 0 -1"/>
-            <limit lower="-0.523598767" upper="0.523598767" effort="1000" velocity="1.0" />
-            <dynamics damping="0.0" friction="2.0"/>
+            <limit lower="-0.698132" upper="0.698132" effort="1000" velocity="1.0" />
+            <dynamics damping="1.0" friction="2.0"/>
         </joint>
         <link name="front_right_wheel_link">
@@ -111,5 +111,5 @@
           <origin xyz="0 0 0" rpy="0 0  0" />
           <axis xyz="0 -1 0"/>
-          <!-- <limit effort="100.0" velocity="10.0"/> -->
+          <limit effort="100.0" velocity="10.0"/>
       </joint>
     </xacro:macro>

File: limo_description/urdf/limo_xacro.xacro (robot description, xacro)
@@ -258,6 +258,5 @@
             <parent link="${parent_prefix}"/>
         </joint>
-        <gazebo reference="${frame_prefix}_link">
-            <material>Gazebo/Yellow</material>
+        <gazebo reference="imu_link">
             <gravity>true</gravity>
             <sensor name="twr_imu" type="imu">

File: limo_description/urdf/properties.xacro (robot description, xacro)
@@ -14,5 +14,4 @@
     <xacro:property name="base_mass" value="2.1557"/>
     <xacro:property name="wheel_mass" value="0.5" />
-    <!-- <xacro:property name="wheel_length" value="0.045" /> -->
     <xacro:property name="wheel_length" value="0.001" />
     <xacro:property name="wheel_radius" value="0.045" />

Commit message: single-mmodel-and-Path Tracking Controller

File: limo_description/urdf/gazbo_control.xacro (robot description, xacro)
@@ -65,6 +65,6 @@
             <command_interface name="velocity"/>
             <command_interface name="position">
-                <param name="min">-0.523598767</param>
-                <param name="max">0.523598767</param>
+                <param name="min">-0.698132</param>
+                <param name="max">0.698132</param>
               </command_interface>
               <state_interface name="position">
@@ -78,4 +78,18 @@
             <command_interface name="velocity"/>
             <command_interface name="position">
+                <param name="min">-0.698132</param>
+                <param name="max">0.698132</param>
+              </command_interface>
+              <state_interface name="position">
+                <param name="initial_value">0.0</param>
+              </state_interface>
+              <state_interface name="velocity">
+              </state_interface>
+              <state_interface name="effort"/>
+        </joint>
+<!--
+        <joint name="main_steering">
+            <command_interface name="velocity"/>
+            <command_interface name="position">
                 <param name="min">-0.523598767</param>
                 <param name="max">0.523598767</param>
@@ -87,24 +101,22 @@
               </state_interface>
               <state_interface name="effort"/>
-        </joint>
+        </joint> -->
     </ros2_control>
     <gazebo reference="base_footprint">
-            <mu1>10</mu1>
-            <mu2>10</mu2>
-            <kp>10000000.0</kp>
-            <kd>1.0</kd>
-            <minDepth>0.01</minDepth>
-            <fdir1>1 0 0</fdir1>
-            <maxContacts value="64"/>
-        </gazebo>
+        <minDepth>0.0002</minDepth>
+        <kp  value="1000000.0"/>
+        <kd  value="100.0"/>
+    </gazebo>
     <gazebo reference="base_link">
-            <mu1>10</mu1>
-            <mu2>10</mu2>
-            <kp>10000000.0</kp>
-            <kd>1.0</kd>
-            <minDepth>0.01</minDepth>
-            <fdir1>1 0 0</fdir1>
-            <maxContacts value="64"/>
-        </gazebo>
+        <minDepth>0.0002</minDepth>
+        <kp  value="1000000.0"/>
+        <kd  value="100.0"/>
+    </gazebo>
+<!--
+    <gazebo reference="main_steering_link">
+        <minDepth>0.0002</minDepth>
+        <kp  value="1000000.0"/>
+        <kd  value="100.0"/>
+    </gazebo> -->
     <gazebo reference="front_left_wheel_link">
         <mu1>10.0</mu1>
@@ -112,5 +124,4 @@
         <minDepth>0.0002</minDepth>
         <kp  value="1000000.0"/>
-        <kd  value="100.0"/>
     </gazebo>
     <gazebo reference="front_right_wheel_link">
@@ -119,5 +130,4 @@
         <minDepth>0.0002</minDepth>
         <kp  value="1000000.0"/>
-        <kd  value="100.0"/>
     </gazebo>
     <gazebo reference="rear_left_wheel_link">
@@ -126,5 +136,4 @@
         <minDepth>0.0002</minDepth>
         <kp  value="1000000.0"/>
-        <kd  value="100.0"/>
     </gazebo>
     <gazebo reference="rear_right_wheel_link">
@@ -133,5 +142,4 @@
         <minDepth>0.0002</minDepth>
         <kp  value="1000000.0"/>
-        <kd  value="100.0"/>
     </gazebo>
 </robot>

File: limo_description/urdf/limo_ackerman.urdf.xacro (robot description, xacro)
@@ -60,4 +60,25 @@
         <origin xyz="${wheelbase/2} ${-track/2} ${wheel_vertical_offset}" rpy="${M_PI} 0 0" />
     </xacro:limo_right_steering_hinge>
+    <!-- <link name="main_steering_link">
+        <inertial>
+            <mass value="0.25" />
+            <inertia ixx="0.00525" ixy="0" ixz="0" iyy="0.00035" iyz="0" izz="0.00525" />
+            <origin xyz="0 0 0" />
+        </inertial>
+        <visual>
+            <origin xyz="0 0 0" rpy="0 0 0" />
+            <geometry>
+                <mesh filename="file://$(find limo_description)/meshes/steering.dae" scale="1 1 1"/>
+            </geometry>
+        </visual>
+    </link>
+    <joint name="main_steering" type="revolute">
+        <parent link="base_link"/>
+        <child link="main_steering_link"/>
+        <origin xyz="${wheelbase/2} 0.0 ${wheel_vertical_offset * -2.0}" rpy="${M_PI} 0 0" />
+        <axis xyz="0 0 -1" />
+        <limit lower="-0.523598767" upper="0.523598767" effort="1000" velocity="10.0" />
+        <dynamics damping="0.0" friction="0.0"/>
+    </joint> -->
     <!-- Back Wheel -->
     <xacro:limo_wheel parent_prefix="base_link" wheel_prefix="rear_left" reflect="1" >

File: limo_description/urdf/limo_steering_hinge.xacro (robot description, xacro)
@@ -28,5 +28,5 @@
             <axis xyz="0 0 1" />
             <limit lower="-0.523598767" upper="0.523598767" effort="1000" velocity="1.0" />
-            <dynamics damping="1.0" friction="2.0"/>
+            <dynamics damping="1.0" friction="0.5"/>
         </joint>
         <link name="${wheel_prefix}_wheel_link">
@@ -55,5 +55,5 @@
           <origin xyz="0 0 0" rpy="0 0  0" />
           <axis xyz="0 1 0"/>
-          <limit effort="100.0" velocity="10.0"/>
+          <!-- <limit effort="100.0" velocity="10.0"/> -->
       </joint>
     </xacro:macro>
@@ -84,5 +84,5 @@
             <axis xyz="0 0 -1"/>
             <limit lower="-0.523598767" upper="0.523598767" effort="1000" velocity="1.0" />
-            <dynamics damping="1.0" friction="2.0"/>
+            <dynamics damping="1.0" friction="0.5"/>
         </joint>
         <link name="front_right_wheel_link">
@@ -111,5 +111,5 @@
           <origin xyz="0 0 0" rpy="0 0  0" />
           <axis xyz="0 -1 0"/>
-          <limit effort="100.0" velocity="10.0"/>
+          <!-- <limit effort="100.0" velocity="10.0"/> -->
       </joint>
     </xacro:macro>

Commit message: uppdate odom scripts

File: limo_description/urdf/gazbo_control.xacro (robot description, xacro)
@@ -6,4 +6,15 @@
         </plugin>
     </gazebo>
+    <!-- <gazebo>
+      <plugin name="ground_truth_plugin" filename="libgazebo_ros_p3d.so">
+        <ros>
+          <namespace>/ground_truth</namespace>
+          <remapping>odom:=pose</remapping>
+        </ros>
+        <body_name>base_footprint</body_name>
+        <frameName>world</frameName>
+        <updateRate>100.0</updateRate>
+      </plugin>
+    </gazebo> -->
     <ros2_control name="GazeboSystem" type="system">
         <hardware>

File: limo_description/urdf/limo_ackerman.urdf.xacro (robot description, xacro)
@@ -44,7 +44,7 @@
         <child link="inertial_link" />
     </joint> -->
-    <xacro:limo_laser parent_prefix="base_link" frame_prefix="laser">
+    <!-- <xacro:limo_laser parent_prefix="base_link" frame_prefix="laser">
         <origin xyz="0.103 0 -0.034" rpy="0 0 0"/>
-    </xacro:limo_laser>
+    </xacro:limo_laser> -->
     <xacro:limo_depth_camera parent_prefix="base_link" frame_prefix="depth_camera">
         <origin xyz="0.084 0 0.026" rpy="0 0 0"/>

File: limo_description/urdf/properties.xacro (robot description, xacro)
@@ -14,5 +14,5 @@
     <xacro:property name="base_mass" value="2.1557"/>
     <xacro:property name="wheel_mass" value="0.5" />
-    <xacro:property name="wheel_length" value="0.001" />
+    <xacro:property name="wheel_length" value="0.01" />
     <xacro:property name="wheel_radius" value="0.045" />
 </robot>

Commit message: update lab1.1

File: limo_description/urdf/gazbo_control.xacro (robot description, xacro)
@@ -12,5 +12,5 @@
           <remapping>odom:=pose</remapping>
         </ros>
-        <body_name>base_footprint</body_name>
+        <body_name>base_link</body_name>
         <frameName>world</frameName>
         <updateRate>100.0</updateRate>
@@ -99,62 +99,74 @@
               <state_interface name="effort"/>
         </joint>
-<!--
-        <joint name="main_steering">
-            <command_interface name="velocity"/>
-            <command_interface name="position">
-                <param name="min">-0.523598767</param>
-                <param name="max">0.523598767</param>
-              </command_interface>
-              <state_interface name="position">
-                <param name="initial_value">0.0</param>
-              </state_interface>
-              <state_interface name="velocity">
-              </state_interface>
-              <state_interface name="effort"/>
-        </joint> -->
     </ros2_control>
-    <gazebo reference="base_footprint">
-        <minDepth>0.0002</minDepth>
-        <kp  value="1000000.0"/>
-        <kd  value="100.0"/>
+    <gazebo>
+        <mu1 value="10"/>
+        <mu2 value="10"/>
+        <kp value="10000000.0" />
+        <kd value="1.0" />
+        <fdir1 value="1 0 0"/>
+        <minDepth value="0.001" />
+        <maxContacts value="64"/>
     </gazebo>
+    <xacro:macro name="limo_wheel_transmission" params="wheel_prefix">
+        <transmission name="${wheel_prefix}_wheel_trans" type="SimpleTransmission">
+            <type>transmission_interface/SimpleTransmission</type>
+            <actuator name="${wheel_prefix}_wheel_motor">
+                <hardwareInterface>hardware_interface/VelocityJointInterface</hardwareInterface>
+            </actuator>
+            <joint name="${wheel_prefix}_wheel">
+                <hardwareInterface>hardware_interface/VelocityJointInterface</hardwareInterface>
+            </joint>
+        </transmission>
+    </xacro:macro>
+    <xacro:macro name="limo_steering_hinge_transmission" params="wheel_prefix">
+        <transmission name="${wheel_prefix}_wheel_trans" type="SimpleTransmission">
+            <type>transmission_interface/SimpleTransmission</type>
+            <actuator name="${wheel_prefix}_wheel_motor">
+                <hardwareInterface>hardware_interface/EffortJointInterface</hardwareInterface>
+            </actuator>
+            <joint name="${wheel_prefix}_wheel">
+                <hardwareInterface>hardware_interface/EffortJointInterface</hardwareInterface>
+            </joint>
+        </transmission>
+    </xacro:macro>
+    <xacro:limo_wheel_transmission wheel_prefix="front_right" />
+    <xacro:limo_wheel_transmission wheel_prefix="front_left" />
+    <xacro:limo_wheel_transmission wheel_prefix="rear_left" />
+    <xacro:limo_wheel_transmission wheel_prefix="rear_right" />
+    <xacro:limo_steering_hinge_transmission wheel_prefix="front_left_steering" />
+    <xacro:limo_steering_hinge_transmission wheel_prefix="front_right_steering" />
     <gazebo reference="base_link">
-        <minDepth>0.0002</minDepth>
-        <kp  value="1000000.0"/>
-        <kd  value="100.0"/>
+        <minDepth>0.001</minDepth>
+        <kp value="10000000.0"/>
+        <kd value="1.0"/>
     </gazebo>
-<!--
-    <gazebo reference="main_steering_link">
-        <minDepth>0.0002</minDepth>
-        <kp  value="1000000.0"/>
-        <kd  value="100.0"/>
-    </gazebo> -->
     <gazebo reference="front_left_wheel_link">
-        <mu1>10.0</mu1>
+       <mu1>10.0</mu1>
         <mu2>10.0</mu2>
-        <minDepth>0.0002</minDepth>
-        <kp  value="1000000.0"/>
-        <kd  value="100.0"/>
+        <minDepth>0.001</minDepth>
+        <kp value="1000000.0"/>
+        <kd value="1.0"/>
     </gazebo>
     <gazebo reference="front_right_wheel_link">
-        <mu1>10.0</mu1>
+       <mu1>10.0</mu1>
         <mu2>10.0</mu2>
-        <minDepth>0.0002</minDepth>
-        <kp  value="1000000.0"/>
-        <kd  value="100.0"/>
+        <minDepth>0.001</minDepth>
+        <kp value="1000000.0"/>
+        <kd value="1.0"/>
     </gazebo>
     <gazebo reference="rear_left_wheel_link">
-        <mu1>10.0</mu1>
+       <mu1>10.0</mu1>
         <mu2>10.0</mu2>
-        <minDepth>0.0002</minDepth>
-        <kp  value="1000000.0"/>
-        <kd  value="100.0"/>
+        <minDepth>0.001</minDepth>
+        <kp value="1000000.0"/>
+        <kd value="1.0"/>
     </gazebo>
     <gazebo reference="rear_right_wheel_link">
-        <mu1>10.0</mu1>
+       <mu1>10.0</mu1>
         <mu2>10.0</mu2>
-        <minDepth>0.0002</minDepth>
-        <kp  value="1000000.0"/>
-        <kd  value="100.0"/>
+        <minDepth>0.001</minDepth>
+        <kp value="1000000.0"/>
+        <kd value="1.0"/>
     </gazebo>
 </robot>

File: limo_description/urdf/limo_ackerman.urdf.xacro (robot description, xacro)
@@ -29,26 +29,10 @@
         <xacro:box_inertial_matrix  m="${base_mass}" w="${base_x_size}" l="${base_y_size}" h="${base_z_size}" />
     </link>
-<!--
-   <link name="inertial_link">
-        <inertial>
-            <origin xyz="0.0 0.0 0.0" />
-            <mass value="${base_mass}" />
-            <inertia ixx="0.0043832566666666675" ixy="0" ixz="0"
-                     iyy="0.004832360833333334" iyz="0"
-                     izz="0.005622784166666667" />
-        </inertial>
-    </link>
-    <joint name="inertial_joint" type="fixed">
-        <origin xyz="0 0 0" rpy="0 0 0" />
-        <parent link="base_link" />
-        <child link="inertial_link" />
-    </joint> -->
-    <!-- <xacro:limo_laser parent_prefix="base_link" frame_prefix="laser">
+    <xacro:limo_laser parent_prefix="base_link" frame_prefix="laser">
         <origin xyz="0.103 0 -0.034" rpy="0 0 0"/>
-    </xacro:limo_laser> -->
-    <!-- <xacro:limo_depth_camera parent_prefix="base_link" frame_prefix="depth_camera">
+    </xacro:limo_laser>
+    <xacro:limo_depth_camera parent_prefix="base_link" frame_prefix="depth_camera">
         <origin xyz="0.084 0 0.026" rpy="0 0 0"/>
     </xacro:limo_depth_camera>
-     -->
     <xacro:limo_imu parent_prefix="base_link" frame_prefix="imu">
         <origin xyz="0.0 0 -0.1" rpy="0 0 0"/>
@@ -61,30 +45,9 @@
         <origin xyz="${wheelbase/2} ${-track/2} ${wheel_vertical_offset}" rpy="${M_PI} 0 0" />
     </xacro:limo_right_steering_hinge>
-    <!-- <link name="main_steering_link">
-        <inertial>
-            <mass value="0.25" />
-            <inertia ixx="0.00525" ixy="0" ixz="0" iyy="0.00035" iyz="0" izz="0.00525" />
-            <origin xyz="0 0 0" />
-        </inertial>
-        <visual>
-            <origin xyz="0 0 0" rpy="0 0 0" />
-            <geometry>
-                <mesh filename="file://$(find limo_description)/meshes/steering.dae" scale="1 1 1"/>
-            </geometry>
-        </visual>
-    </link>
-    <joint name="main_steering" type="revolute">
-        <parent link="base_link"/>
-        <child link="main_steering_link"/>
-        <origin xyz="${wheelbase/2} 0.0 ${wheel_vertical_offset * -2.0}" rpy="${M_PI} 0 0" />
-        <axis xyz="0 0 -1" />
-        <limit lower="-0.523598767" upper="0.523598767" effort="1000" velocity="10.0" />
-        <dynamics damping="0.0" friction="0.0"/>
-    </joint> -->
     <!-- Back Wheel -->
-    <xacro:limo_wheel parent_prefix="base_link" wheel_prefix="rear_left" reflect="1" >
+    <xacro:limo_wheel parent_prefix="base_link" wheel_prefix="rear_left" reflect="1" fixed_on="false">
         <origin xyz="${-wheelbase/2} ${track/2} ${wheel_vertical_offset}" rpy="0 0 0" />
     </xacro:limo_wheel>
-    <xacro:limo_wheel parent_prefix="base_link" wheel_prefix="rear_right" reflect="-1">
+    <xacro:limo_wheel parent_prefix="base_link" wheel_prefix="rear_right" reflect="-1" fixed_on="false">
         <origin xyz="${-wheelbase/2} ${-track/2} ${wheel_vertical_offset}" rpy="${M_PI} 0 0" />
     </xacro:limo_wheel>

File: limo_description/urdf/limo_xacro.xacro (robot description, xacro)
@@ -1,11 +1,11 @@
 <?xml version="1.0"?>
 <robot name="limo_xacro" xmlns:xacro="http://ros.org/wiki/xacro">
-    <!-- <xacro:macro name="limo_wheel" params="parent_prefix wheel_prefix reflect *joint_pose visual_on:=true fixed_on:=false">
+    <xacro:macro name="limo_wheel" params="parent_prefix wheel_prefix reflect *joint_pose visual_on:=true fixed_on:=false">
         <link name="${wheel_prefix}_wheel_link">
-            <inertial>
+            <!-- <inertial>
                 <origin xyz="0 ${wheel_length/2} 0" rpy="1.57 0 0" />
                 <mass value="0.5" />
                 <inertia ixx="0.00033749999999999996" ixy="0" ixz="0" iyy="0.00033749999999999996" iyz="0" izz="0.00050625" />
-            </inertial>
+            </inertial> -->
             <xacro:if value="${visual_on}">
                 <visual>
@@ -22,7 +22,7 @@
               </geometry>
             </collision>
-        </link> -->
-        <!-- Conditionally set the joint type -->
-        <!-- <xacro:if value="${fixed_on}">
+            <xacro:cylinder_inertial_matrix  m="${wheel_mass}" r="${wheel_radius}"  h="${wheel_length}" />
+        </link>
+        <xacro:if value="${fixed_on}">
             <joint name="${wheel_prefix}_wheel" type="fixed">
                 <parent link="${parent_prefix}"/>
@@ -40,16 +40,16 @@
             </joint>
         </xacro:unless>
-    </xacro:macro> -->
-    <xacro:macro name="limo_wheel" params="parent_prefix wheel_prefix reflect *joint_pose">
+    </xacro:macro>
+    <!-- <xacro:macro name="limo_wheel" params="parent_prefix wheel_prefix reflect *joint_pose">
         <link name="${wheel_prefix}_wheel_link">
-            <!-- <inertial>
+            <inertial>
                 <origin xyz="0 0 0" />
                 <mass value="0.5" />
                 <inertia ixx="0.01055" ixy="0" ixz="0" iyy="0.00075" iyz="0" izz="0.01055" />
-            </inertial> -->
+            </inertial>
             <visual>
                 <origin xyz="0 0 0" rpy="0 0 0" />
                 <geometry>
-                    <mesh filename="file://$(find limo_description)/meshes/limo_optimal_wheels.dae" />
+                    <mesh filename="file://$(find limo_description)/meshes/limo_wheel.dae" />
                 </geometry>
             </visual>
@@ -68,5 +68,5 @@
             <axis xyz="0 ${reflect*1} 0"/>
         </joint>
-    </xacro:macro>
+    </xacro:macro> -->
     <xacro:macro name="limo_laser" params="parent_prefix frame_prefix *joint_pose">
         <link name='${frame_prefix}_link'>

File: limo_description/urdf/properties.xacro (robot description, xacro)
@@ -11,8 +11,8 @@
     <!-- <xacro:property name="track" value="0.14"/> -->
     <xacro:property name="track" value="0.13"/>
-    <xacro:property name="wheel_vertical_offset" value="-0.100998" />
+    <xacro:property name="wheel_vertical_offset" value="-0.10" />
     <xacro:property name="base_mass" value="2.1557"/>
-    <xacro:property name="wheel_mass" value="0.5" />
-    <xacro:property name="wheel_length" value="0.01" />
+    <xacro:property name="wheel_mass" value="0.25" />
+    <xacro:property name="wheel_length" value="0.001" />
     <xacro:property name="wheel_radius" value="0.045" />
 </robot>
